File: KiCad/2018-03-08 Intercourse/2018-03-08 Intercourse 01.kicad_pcb (KiCad board)
At the start: 2 copper layers, 46 parts, among them J1 USB_C_Receptacle, J2 TP_RST, J3 TP_TX, J4 TP_RX, J5 TP_GPIO0, J6 TP_GND1, J7 TP_GND2, U1 LTC3225, U2 TPS61221DCKR, U3 W25Q32FVSSIG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

Commit message: backup of layouting process
Parts:
- U2: footprint TO_SOT_Packages_SMD:SC-70-8_Handsoldering -> sc_70-6:sc_70-6
- moved Y1 74.4 mm to (188.0, 83.8)
- moved R4 66.4 mm to (168.9, 102.9), turned to 180 degrees
- moved R5 61.7 mm to (172.4, 101.6), turned to 90 degrees
- moved R6 59.4 mm to (163.8, 71.1)
- moved C10 54.7 mm to (169.2, 78.7), turned to 180 degrees
- moved R7 50.9 mm to (162.6, 95.2), turned to 90 degrees
- moved C1 49.9 mm to (127.0, 85.1), turned to 90 degrees
- moved C8 46.3 mm to (168.9, 100.3)
- moved U4 45.0 mm to (162.6, 85.1), turned to 270 degrees
- moved C12 42.7 mm to (155.9, 78.1)
- moved J1 39.2 mm to (115.4, 101.6), turned to 270 degrees
- moved R15 37.5 mm to (148.5, 121.9)
- moved C11 37.3 mm to (148.6, 106.7)
- moved R13 37.3 mm to (148.5, 111.8)
- moved C9 37.2 mm to (161.0, 78.1)
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Other:
- board outline added: 85.6 x 54 mm

Commit message: backup pcb layout
Parts:
- moved R15 38.2 mm to (156.2, 84.5), turned to 180 degrees
- moved R2 30.5 mm to (156.2, 99.0)
- moved R3 30.5 mm to (156.2, 104.2)
- moved R14 28.4 mm to (156.2, 89.5), turned to 180 degrees
- moved R13 25.9 mm to (156.2, 87.0), turned to 180 degrees
- moved C11 25.9 mm to (156.2, 81.9), turned to 180 degrees
- moved Y1 19.1 mm to (168.9, 85.7), turned to 180 degrees
- moved C7 14.5 mm to (168.9, 88.9), turned to 0 degrees
- moved C2 13.3 mm to (146.2, 99.1)
- moved L1 13.3 mm to (150.7, 100.4)
- moved C4 13.3 mm to (146.2, 104.2)
- moved U2 13.3 mm to (146.9, 101.7)
- moved C9 8.55 mm to (168.9, 81.3)
- moved R6 7.65 mm to (164.5, 78.7), turned to 270 degrees
- moved R10 6.71 mm to (80.0, 95.9)
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
Commit message: advanced layout, backuping
Parts:
- moved D5 106.9 mm to (186.7, 115.6)
- moved R12 106.8 mm to (186.7, 113.0)
- moved D4 99.8 mm to (179.1, 115.6)
- moved R11 99.7 mm to (179.1, 113.0)
- moved D3 93.2 mm to (171.4, 115.6)
- moved R10 93.0 mm to (171.4, 113.0)
- moved D2 87.1 mm to (163.8, 115.6)
- moved R9 86.9 mm to (163.8, 113.0)
- moved D1 81.6 mm to (156.2, 115.6)
- moved R8 81.4 mm to (156.2, 113.0)
- moved J5 35.6 mm to (139.7, 97.8)
- moved R3 9.92 mm to (153.8, 94.6), turned to 0 degrees
- moved R2 8.85 mm to (148.5, 94.6), turned to 180 degrees
- moved C4 8.41 mm to (154.6, 103.6), turned to 270 degrees
- moved C2 5.54 mm to (149.5, 103.6), turned to 270 degrees
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
Commit message: ready to route
Parts:
- added J8: TP_GND3, C_Connectors:C_Connector_2mm, F.Cu at (176.5, 97.2)
- J5: footprint C_Connectors:C_Connector_2mm -> Measurement_Points:Measurement_Point_Round-SMD-Pad_Small
- moved J5 25.2 mm to (156.2, 78.7)
- moved J6 12.2 mm to (190.5, 106.0)
- moved J4 10.8 mm to (185.4, 97.2)
- moved J3 2.62 mm to (185.4, 106.0)
- moved J2 1.42 mm to (176.5, 106.0)
- moved J7 0.64 mm to (190.5, 97.2)
Changed lines of the file:
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@@
 (kicad_pcb (version 4) (host pcbnew 4.0.7)
   (general
-    (links 106)
-    (no_connects 106)
+    (links 107)
+    (no_connects 107)
     (area 109.549999 74.559999 195.250001 128.640001)
     (thickness 1.6)
@@
     (tracks 0)
     (zones 0)
-    (modules 46)
+    (modules 47)
     (nets 61)
   )
@@
   )
   (module C_Connectors:C_Connector_2mm (layer F.Cu)
-    (at 175.26 106.68)
-    (fp_text reference J2 (at 0 2.54) (layer F.SilkS)
+    (at 176.53 106.045)
+    (fp_text reference J2 (at 0 -3.175) (layer F.SilkS)
       (effects (font (size 1 1) (thickness 0.15)))
     )
@@
   )
   (module C_Connectors:C_Connector_2mm (layer F.Cu)
-    (at 182.88 106.68)
-    (fp_text reference J3 (at 0 2.54) (layer F.SilkS)
+    (at 185.42 106.045)
+    (fp_text reference J3 (at 0 -3.175) (layer F.SilkS)
       (effects (font (size 1 1) (thickness 0.15)))
     )
@@
   )
   (module C_Connectors:C_Connector_2mm (layer F.Cu)
-    (at 190.5 106.68)
-    (fp_text reference J4 (at 0 2.54) (layer F.SilkS)
+    (at 185.42 97.155)
+    (fp_text reference J4 (at 0 3.175) (layer F.SilkS)
       (effects (font (size 1 1) (thickness 0.15)))
     )
@@
   )
   (module C_Connectors:C_Connector_2mm (layer F.Cu)
-    (at 139.7 97.79)
-    (fp_text reference J5 (at 0 2.54) (layer F.SilkS)
-      (effects (font (size 1 1) (thickness 0.15)))
-    )
-    (fp_text value TP_GPIO0 (at 0 -2.54) (layer F.Fab)
+    (at 190.5 106.045)
+    (fp_text reference J6 (at 0 -3.175) (layer F.SilkS)
+      (effects (font (size 1 1) (thickness 0.15)))
+    )
+    (fp_text value TP_GND1 (at 0 -2.54) (layer F.Fab)
       (effects (font (size 1 1) (thickness 0.15)))
     )
     (pad 1 thru_hole circle (at 0 0) (size 2.5 2.5) (drill 2) (layers *.Cu *.Mask)
-      (net 40 MODE))
+      (net 4 GND))
   )
   (module C_Connectors:C_Connector_2mm (layer F.Cu)
-    (at 182.88 96.52)
-    (fp_text reference J6 (at 0 2.54) (layer F.SilkS)
-      (effects (font (size 1 1) (thickness 0.15)))
-    )
-    (fp_text value TP_GND1 (at 0 -2.54) (layer F.Fab)
-      (effects (font (size 1 1) (thickness 0.15)))
-    )
-    (pad 1 thru_hole circle (at 0 0) (size 2.5 2.5) (drill 2) (layers *.Cu *.Mask)
-      (net 4 GND))
-  )
-  (module C_Connectors:C_Connector_2mm (layer F.Cu)
-    (at 190.5 96.52)
-    (fp_text reference J7 (at 0 2.54) (layer F.SilkS)
+    (at 190.5 97.155)
+    (fp_text reference J7 (at 0 3.175) (layer F.SilkS)
       (effects (font (size 1 1) (thickness 0.15)))
     )
@@
     )
   )
+  (module C_Connectors:C_Connector_2mm (layer F.Cu)
+    (at 176.53 97.155)
+    (fp_text reference J8 (at 0 3.175) (layer F.SilkS)
+      (effects (font (size 1 1) (thickness 0.15)))
+    )
+    (fp_text value TP_GND3 (at 0 -2.54) (layer F.Fab)
+      (effects (font (size 1 1) (thickness 0.15)))
+    )
+    (pad 1 thru_hole circle (at 0 0) (size 2.5 2.5) (drill 2) (layers *.Cu *.Mask)
+      (net 4 GND))
+  )
+  (module Measurement_Points:Measurement_Point_Round-SMD-Pad_Small (layer F.Cu)
+    (at 156.21 78.74)
+    (descr "Mesurement Point, Round, SMD Pad, DM 1.5mm,")
+    (tags "Mesurement Point Round SMD Pad 1.5mm")
+    (attr virtual)
+    (fp_text reference J5 (at 0 -2) (layer F.SilkS)
+      (effects (font (size 1 1) (thickness 0.15)))
+    )
+    (fp_text value TP_GPIO0 (at 0 2) (layer F.Fab)
+      (effects (font (size 1 1) (thickness 0.15)))
+    )
+    (fp_circle (center 0 0) (end 1 0) (layer F.CrtYd) (width 0.05))
+    (pad 1 smd circle (at 0 0) (size 1.5 1.5) (layers F.Cu F.Mask)
+      (net 40 MODE))
+  )
   (gr_line (start 121.30625 74.61) (end 122.55 74.61) (layer Edge.Cuts) (width 0.1))

Commit message: layout 01 before drc
Parts:
- moved J3 8.89 mm to (185.4, 97.2)
- moved J4 8.89 mm to (185.4, 106.0)
- moved C9 1.31 mm to (168.6, 82.5), turned to 180 degrees
- moved R7 0.16 mm to (162.6, 95.3)
Routing:
- net GND: track 0.00 -> 374.1 mm, vias 0 -> 4
- net VDD: track 0.00 -> 91.6 mm, vias 0 -> 2
- net VBUS: track 0.00 -> 90.4 mm, vias 0 -> 4
- net Net-(C1-Pad1): track 0.00 -> 58.9 mm
- net CHARGE_LED: track 0.00 -> 57.4 mm, vias 0 -> 2
- net Net-(R12-Pad1): track 0.00 -> 46.3 mm, vias 0 -> 2
- net Net-(R9-Pad1): track 0.00 -> 43.3 mm, vias 0 -> 2
- net Net-(R11-Pad1): track 0.00 -> 42.2 mm, vias 0 -> 2
- net Net-(R10-Pad1): track 0.00 -> 40.9 mm, vias 0 -> 2
- net RST: track 0.00 -> 36.3 mm, vias 0 -> 2
- net Net-(J4-Pad1): track 0.00 -> 32.0 mm, vias 0 -> 2
- net USB_PWR: track 0.00 -> 27.0 mm, vias 0 -> 2
- net Net-(J3-Pad1): track 0.00 -> 26.4 mm, vias 0 -> 2
- net Net-(C1-Pad2): track 0.00 -> 24.3 mm
- net Net-(J1-PadS1): track 0.00 -> 21.2 mm, vias 0 -> 2
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Other:
- rule trace_min: 0.2 -> 0.15

Commit message: drc complete
Parts:
- moved R5 0.27 mm to (172.7, 101.6)
Routing:
- net GND: track 374.1 -> 393.3 mm, vias 4 -> 9
- net Net-(U3-Pad2): track 19.6 -> 23.4 mm
- net CHARGE_LED: track 57.4 -> 58.4 mm
- net Net-(R6-Pad2): track 9.87 -> 9.09 mm
- net Net-(R9-Pad1): track 43.3 -> 43.9 mm
- net Net-(R10-Pad1): track 40.9 -> 41.4 mm

Commit message: created graphic layout and edited it into pcb
Parts:
- added G***: LOGO, shapes:layout_02, F.Cu at (152.4, 102.4)
- added G***: LOGO, shapes:layout_02_back, B.Cu at (144.8, 101.6)
Routing:
- net Net-(C1-Pad1): track 58.9 -> 50.8 mm
- net (no net): track 0.00 -> 8.04 mm
- added copper zone on F.Cu, net (none)
- added copper zone on F.Cu, net GND
